File: chapters/kicad/Elektronika/Elektronika.kicad_sch (KiCad schematic)
At the start: 5 parts, among them SW1 SW_DPST_x2

Commit message: vprašanja
Parts:
- SW1: value SW_DPST_x2 -> S
Changed lines of the file:
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@@
 			)
 		)
-		(property "Value" "SW_DPST_x2"
+		(property "Value" "S"
 			(at 118.11 80.01 0)
-			(hide yes)
 			(show_name no)
 			(do_not_autoplace no)
